File: the_main_pcb/the_main_pcb.kicad_pcb (KiCad board)
At the start: 2 copper layers, 1 part

Commit message: worked more on the pcb
Parts:
- added D1: LED, LED_THT:LED_D1.8mm_W3.3mm_H2.4mm, F.Cu at (120.1, 57.9)
- added J1: Conn_01x02_Pin, Connector_PinHeader_2.54mm:PinHeader_1x02_P2.54mm_Vertical, F.Cu at (163.0, 51.1)
- added R1: 330, Resistor_THT:R_Axial_DIN0309_L9.0mm_D3.2mm_P12.70mm_Horizontal, F.Cu at (120.0, 64.3)
- added R2: R_Photo, LED_THT:LED_D1.8mm_W3.3mm_H2.4mm, F.Cu at (114.4, 58.8)
- added R3: 10K, Resistor_THT:R_Axial_DIN0309_L9.0mm_D3.2mm_P12.70mm_Horizontal, F.Cu at (141.6, 86.3)
- U1: value ~ -> esp32
- moved U1 46.6 mm to (143.6, 68.6)
Connections:
- U1 pad 1: unconnected-(U1-3.3-Pad1) -> 3V3
- U1 pad 15: unconnected-(U1-D23-Pad15) -> R1
- U1 pad 16: unconnected-(U1-VIN-Pad16) -> Net-(J1-Pin_1)
- U1 pad 17: unconnected-(U1-GND-Pad17) -> Net-(J1-Pin_2)
- U1 pad 2: unconnected-(U1-GND-Pad2) -> GND
- U1 pad 27: unconnected-(U1-D34-Pad27) -> LDR
Routing:
- net LDR: track 0.00 -> 67.9 mm
- net GND: track 0.00 -> 37.3 mm
- net 3V3: track 0.00 -> 19.2 mm
- net R1: track 0.00 -> 12.9 mm
- net Net-(J1-Pin_2): track 0.00 -> 7.55 mm
- net Net-(J1-Pin_1): track 0.00 -> 7.55 mm
- net Net-(D1-A): track 0.00 -> 3.87 mm
Other:
- board text added: "esp32"

Commit message: start working on the 3D
Other:
- board outline added: 60 x 55.9 mm
Changed lines of the file:
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@@
 		(embedded_fonts no)
 	)
+	(gr_rect
+		(start 110.4 42.1)
+		(end 170.4 98)
+		(stroke
+			(width 0.1)
+			(type solid)
+		)
+		(fill no)
+		(layer "Edge.Cuts")
+	)
 	(gr_text "esp32"
-		(at 141 57.9 0)
+		(at 146.3 56.5 0)
 		(layer "F.Cu")
 		(effects
@@
 				(bold yes)
 			)
-			(justify left bottom)
+			(justify left bottom mirror)
 		)
 	)

Commit message: updated the PCB pdf
Parts:
- added D2: LED, LED_THT:LED_D1.8mm_W3.3mm_H2.4mm, F.Cu at (109.2, 74.7)
- moved R2 8.95 mm to (105.5, 57.9)
Routing:
- net GND: track 37.3 -> 62.2 mm
- net Net-(D1-A): track 3.87 -> 23.0 mm
- net LDR: track 67.9 -> 80.1 mm
- net 3V3: track 19.2 -> 25.9 mm
Other:
- board size 60 x 55.9 mm -> 71.3 x 55.9 mm
