File: the_main_pcb/the_main_pcb.kicad_sch (KiCad schematic)
At the start: 0 parts

Commit message: done with the esp32 costume pcb
Parts:
- added U1: ~, esp32_footprint:Untitled, symbol esp32:esp32
Changed lines of the file:
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@@
 	(generator_version "9.0")
 	(paper "A4")
+	(symbol
+		(lib_id "esp32:esp32")
+		(at 123.19 80.01 0)
+		(unit 1)
+		(exclude_from_sim no)
+		(in_bom yes)
+		(on_board yes)
+		(dnp no)
+		(fields_autoplaced yes)
+		(property "Reference" "U1"
+			(at 123.19 62.23 0)
+			(effects
+				(font
+					(size 1.27 1.27)
+				)
+			)
+		)
+		(property "Value" "~"
+			(at 123.19 64.77 0)
+			(effects
+				(font
+					(size 1.27 1.27)
+				)
+			)
+		)
+		(property "Footprint" "esp32_footprint:Untitled"
+			(at 123.19 80.01 0)
+			(effects
+				(font
+					(size 1.27 1.27)
+				)
+				(hide yes)
+			)
+		)
+		(property "Datasheet" ""
+			(at 123.19 80.01 0)
+			(effects
+				(font
+					(size 1.27 1.27)
+				)
+				(hide yes)
+			)
+		)
+		(property "Description" ""
+			(at 123.19 80.01 0)
+			(effects
+				(font
+					(size 1.27 1.27)
+				)
+				(hide yes)
+			)
+		)
+		(pin "29"
+		)
+		(pin "11"
+		)
+		(pin "21"
+		)
+		(pin "9"
+		)
+		(pin "10"
+		)
+		(pin "22"
+		)
+		(pin "8"
+		)
+		(pin "16"
+		)
+		(pin "13"
+		)
+		(pin "17"
+		)
+		(pin "14"
+		)
+		(pin "15"
+		)
+		(pin "26"
+		)
+		(pin "28"
+		)
+		(pin "6"
+		)
+		(pin "5"
+		)
+		(pin "4"
+		)
+		(pin "20"
+		)
+		(pin "27"
+		)
+		(pin "24"
+		)
+		(pin "2"
+		)
+		(pin "1"
+		)
+		(pin "3"
+		)
+		(pin "30"
+		)
+		(pin "25"
+		)
+		(pin "19"
+		)
+		(pin "18"
+		)
+		(pin "23"
+		)
+		(pin "12"
+		)
+		(pin "7"
+		)
+		(instances
+			(project ""
+				(path "/d402f5bd-ed8e-4851-8b19-b2cff888d33d"
+					(reference "U1")
+					(unit 1)
+				)
+			)
+		)
+	)
 	(sheet_instances
 		(path "/"

Commit message: worked more on the pcb
Parts:
- added D1: LED, LED_THT:LED_D1.8mm_W3.3mm_H2.4mm, symbol Device:LED
- added J1: Conn_01x02_Pin, Connector_PinHeader_2.54mm:PinHeader_1x02_P2.54mm_Vertical, symbol Connector:Conn_01x02_Pin
- added R1: 330, Resistor_THT:R_Axial_DIN0309_L9.0mm_D3.2mm_P12.70mm_Horizontal, symbol Device:R
- added R2: R_Photo, LED_THT:LED_D1.8mm_W3.3mm_H2.4mm, symbol Device:R_Photo
- added R3: 10K, Resistor_THT:R_Axial_DIN0309_L9.0mm_D3.2mm_P12.70mm_Horizontal, symbol Device:R
- U1: value ~ -> esp32
Connections:
- net 3V3: now reaches U1.1 (3V3)
- net 3V3: now also R2.1
- net R1: now reaches U1.15 (D23)
- net R1: now also R1.2
- net at U1.16 (VIN): now also J1.1 (Pin_1)
- net at U1.17 (GND): now also J1.2 (Pin_2)
- net GND: now reaches U1.2 (GND)
- net GND: now also D1.1 (K), R3.2
- net LDR: now reaches U1.27 (D34)
- net LDR: now also R2.2, R3.1
- new net: D1.2 (A), R1.1
- no-connect marks 0 -> 24

Commit message: updated the PCB pdf
Parts:
- added D2: LED, LED_THT:LED_D1.8mm_W3.3mm_H2.4mm, symbol Device:LED
Connections:
- net GND: now also D2.1 (K)
- net at D1.2 (A), R1.1: now also D2.2 (A)
Changed lines of the file:
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@@
 	(paper "A4")
+	(junction
+		(at 66.04 95.25)
+		(diameter 0)
+		(color 0 0 0 0)
+	)
 	(junction
 		(at 74.93 110.49)
@@
 		(color 0 0 0 0)
 	)
+	(junction
+		(at 73.66 95.25)
+		(diameter 0)
+		(color 0 0 0 0)
+	)
 	(no_connect
 		(at 135.89 102.87)
@@
 	(wire
 		(pts
+			(xy 66.04 83.82) (xy 66.04 95.25)
+		)
+		(stroke
+			(width 0)
+			(type default)
+		)
+	)
+	(wire
+		(pts
 			(xy 74.93 110.49) (xy 78.74 110.49)
 		)
@@
 		(pts
 			(xy 60.96 95.25) (xy 66.04 95.25)
+		)
+		(stroke
+			(width 0)
+			(type default)
+		)
+	)
+	(wire
+		(pts
+			(xy 73.66 83.82) (xy 73.66 95.25)
 		)
 		(stroke
@@
 					(unit 1)
 				)
+			)
+		)
+	)
+	(symbol
+		(lib_id "Device:LED")
+		(at 69.85 83.82 0)
+		(unit 1)
+		(exclude_from_sim no)
+		(in_bom yes)
+		(on_board yes)
+		(dnp no)
+		(fields_autoplaced yes)
+		(property "Reference" "D2"
+			(at 68.2625 77.47 0)
+			(effects
+				(font
+					(size 1.27 1.27)
+				)
+			)
+		)
+		(property "Value" "LED"
+			(at 68.2625 80.01 0)
+			(effects
+				(font
+					(size 1.27 1.27)
+				)
+			)
+		)
+		(property "Footprint" "LED_THT:LED_D1.8mm_W3.3mm_H2.4mm"
+			(at 69.85 83.82 0)
+			(effects
+				(font
+					(size 1.27 1.27)
+				)
+				(hide yes)
+			)
+		)
+		(property "Datasheet" "~"
+			(at 69.85 83.82 0)
+			(effects
+				(font
+					(size 1.27 1.27)
+				)
+				(hide yes)
+			)
+		)
+		(property "Description" "Light emitting diode"
+			(at 69.85 83.82 0)
+			(effects
+				(font
+					(size 1.27 1.27)
+				)
+				(hide yes)
+			)
+		)
+		(property "Sim.Pins" "1=K 2=A"
+			(at 69.85 83.82 0)
+			(effects
+				(font
+					(size 1.27 1.27)
+				)
+				(hide yes)
+			)
+		)
+		(pin "2"
+		)
+		(pin "1"
+		)
+		(instances
+			(project "the_main_pcb"
+				(path "/d402f5bd-ed8e-4851-8b19-b2cff888d33d"
+					(reference "D2")
+					(unit 1)
+				)
